Commit message: feat(robots_description): Add and update URDF models

File: robots_description/mycobot_pro_450_description/urdf/mycobot_pro_450.urdf (robot description, URDF)
Before this commit: robot mycobot_pro450, 7 links, 6 joints
Links:
- removed link base
- added link base_link, mass 2.0381; collision mesh filename=package://mycobot_pro_450_description/meshes/base.STL; visual mesh filename=package://mycobot_pro_450_description/meshes/base.STL
- link Link1: geometry collision mesh filename=package://mycobot_pro_450_description/meshes/Link1.STL; visual mesh filename=package://mycobot_pro_450_description/meshes/Link1.STL
- link Link2: geometry collision mesh filename=package://mycobot_pro_450_description/meshes/Link2.STL; visual mesh filename=package://mycobot_pro_450_description/meshes/Link2.STL
- link Link3: geometry collision mesh filename=package://mycobot_pro_450_description/meshes/Link3.STL; visual mesh filename=package://mycobot_pro_450_description/meshes/Link3.STL
- link Link4: geometry collision mesh filename=package://mycobot_pro_450_description/meshes/Link4.STL; visual mesh filename=package://mycobot_pro_450_description/meshes/Link4.STL
- link Link5: geometry collision mesh filename=package://mycobot_pro_450_description/meshes/Link5.STL; visual mesh filename=package://mycobot_pro_450_description/meshes/Link5.STL
- link Link6: geometry collision mesh filename=package://mycobot_pro_450_description/meshes/Link6.STL; visual mesh filename=package://mycobot_pro_450_description/meshes/Link6.STL
Joints:
- joint joint1: parent base -> base_link

Commit message: fix(robots_description): Fix the coordinate systems of the URDF robotic arm

File: robots_description/mycobot_pro_450_description/urdf/mycobot_pro_450.urdf (robot description, URDF)
Before this commit: robot mycobot_pro450, 7 links, 6 joints
Links:
- link Link1: mass 0.5442 -> 0.7923
- link Link2: mass 0.58911 -> 0.8204
- link Link3: mass 0.68875 -> 0.6
- link Link4: mass 0.55433 -> 0.4483
- link Link5: mass 0.53025 -> 0.4642
- link Link6: mass 0.10905 -> 0.129
- link base_link: mass 2.0381 -> 2.2569; geometry collision mesh filename=package://mycobot_pro_450_description/meshes/base_link.STL; visual mesh filename=package://mycobot_pro_450_description/meshes/base_link.STL
Joints:
- joint joint1: limit lower=-2.8274 upper=2.8274 effort=100000 velocity=3.7909 -> lower=-2.88 upper=2.88 effort=0 velocity=0; origin xyz=-0.00093304 0 0.17372 rpy=0 0 0 -> xyz=0 0 0.210000000061212 rpy=0 0 0
- joint joint2: axis 0 -1 0 -> 0 0 1; limit lower=-2.1817 upper=2.1817 effort=100000 velocity=3.7909 -> lower=-2.04 upper=2.04 effort=0 velocity=0; origin xyz=0.00017155 -0.072764 0.037522 rpy=0 0 0.00011694 -> xyz=0 0 0 rpy=1.57079632679529 1.5707963267949 0
- joint joint3: axis 0 -1 0 -> 0 0 1; limit lower=-2.687807 upper=2.687807 effort=100000 velocity=3.11 -> lower=-2.74 upper=2.74 effort=0 velocity=0; origin xyz=-0.00011952 0.0394 0.18008 rpy=0 0 0 -> xyz=-0.179219598097142 0 0 rpy=0 0 0
- joint joint4: axis 0 -1 0 -> 0 0 1; limit lower=-2.8274 upper=2.8274 effort=100000 velocity=3.11 -> lower=-2.88 upper=2.88 effort=0 velocity=0; origin xyz=0 -0.027001 0.173 rpy=0 0 0 -> xyz=-0.173780401902847 0 0.0854905429592015 rpy=0 0 -1.5707963267949
- joint joint5: limit lower=-2.8274 upper=2.8274 effort=100000 velocity=3.11 -> lower=-2.88 upper=2.88 effort=0 velocity=0; origin xyz=-1.3818E-05 -0.025698 0.070501 rpy=0 0 -0.00011694 -> xyz=0 -0.097501 0 rpy=1.5708 -1.5708 0
- joint joint6: axis 1 0 0 -> 0 0 1; limit lower=-2.879793 upper=2.879793 effort=100000 velocity=3.11 -> lower=-2.93 upper=2.93 effort=0 velocity=0; origin xyz=0.031841 0.0001386 0.026584 rpy=0 0 0.00011694 -> xyz=0 0.063173 0.00020984 rpy=-1.5708 0 0

File: robots_description/mygripper_f100_description/urdf/mygripper_f100.urdf (robot description, URDF)
Before this commit: robot 3.6, 7 links, 6 joints
Links:
- removed link SL_Link
- removed link SR_Link
- removed link base_link
- added link SL_L_Link, mass 0.006; collision mesh filename=package://mygripper_f100_description/meshes/SL_L_Link.STL; visual mesh filename=package://mygripper_f100_description/meshes/SL_L_Link.STL
- added link SL_R_Link, mass 0.006; collision mesh filename=package://mygripper_f100_description/meshes/SL_R_Link.STL; visual mesh filename=package://mygripper_f100_description/meshes/SL_R_Link.STL
- added link f100_base_link, mass 0.251; collision mesh filename=package://mygripper_f100_description/meshes/f100_base_link.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; visual mesh filename=package://mygripper_f100_description/meshes/f100_base_link.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
- link J2_L_Link: mass 0.0106787406466507 -> 0.015
- link J2_R_Link: mass 0.0106787331581622 -> 0.013
- link J3_L_Link: mass 0.0122763514806654 -> 0.017
- link J3_R_Link: mass 0.0122762764991077 -> 0.018
Joints:
- removed joint J2_R_Joint
- removed joint J3_R_Joint
- removed joint SR_Joint
- added joint J2_R_joint: type revolute, parent f100_base_link, child J2_R_Link, origin xyz=0.056064 -0.019509 0 rpy=0 0 0, axis 0 0 -1, limit lower=-1.012 upper=1.012 effort=0 velocity=0, mimic joint=J2_L_Joint multiplier=-1 offset=0
- added joint J3_R_joint: type revolute, parent J2_R_Link, child J3_R_Link, origin xyz=0.06 0.009756 0 rpy=0 0 0, axis 0 0 -1, limit lower=-1.012 upper=1.012 effort=0 velocity=0, mimic joint=J2_L_Joint multiplier=1 offset=0
- added joint SL_R_joint: type revolute, parent f100_base_link, child SL_R_Link, origin xyz=0.033748 -0.045581 0 rpy=0 0 0, axis 0 0 -1, limit lower=-1.012 upper=1.012 effort=0 velocity=0, mimic joint=J2_L_Joint multiplier=-1 offset=0
- joint J2_L_Joint: origin xyz=-0.00199539964651109 0.0170897105451218 0 rpy=0 0 -0.161189635313468 -> xyz=0.056064 0.017111 0 rpy=0 0 0.00036257; parent base_link -> f100_base_link
- joint J3_L_Joint: origin xyz=0.0607879914104711 0 -0.000499999999989536 rpy=0 0 -0.70066916574601 -> xyz=0.059996 -0.0097778 -0.0005 rpy=0 0 0
- joint SL_Joint: child SL_Link -> SL_L_Link; origin xyz=-0.0243107456319108 0.0431815900188018 0 rpy=0 0 -0.162249613278239 -> xyz=0.033748 0.043203 0 rpy=0 0 0.00036257; parent base_link -> f100_base_link

Commit message: fix(robots_description): Modify the URDF file and add the 450USD file

File: robots_description/mycobot_pro_450_description/urdf/mycobot_pro_450.urdf (robot description, URDF)
Before this commit: robot mycobot_pro450, 7 links, 6 joints
Joints:
- joint joint1: limit lower=-2.88 upper=2.88 effort=0 velocity=0 -> lower=-2.827433 upper=2.82743 effort=0 velocity=2.6178
- joint joint2: limit lower=-2.04 upper=2.04 effort=0 velocity=0 -> lower=-2.181622 upper=2.181622 effort=0 velocity=2.6178
- joint joint3: limit lower=-2.74 upper=2.74 effort=0 velocity=0 -> lower=-2.687807 upper=2.687807 effort=0 velocity=2.6178
- joint joint4: limit lower=-2.88 upper=2.88 effort=0 velocity=0 -> lower=-2.827433 upper=2.827433 effort=0 velocity=2.6178
- joint joint5: limit lower=-2.88 upper=2.88 effort=0 velocity=0 -> lower=-2.827433 upper=2.827433 effort=0 velocity=2.6178
- joint joint6: limit lower=-2.93 upper=2.93 effort=0 velocity=0 -> lower=-2.879793 upper=2.879793 effort=0 velocity=2.6178
