Commit message: fix(USD):Fixed the f100's root joint property

File: robots_description/mygripper_f100_description/urdf/mygripper_f100.urdf (robot description, URDF)
Before this commit: robot mygripper_f100, 7 links, 6 joints
Links:
- removed link J2_L_Link
- removed link J2_R_Link
- removed link J3_L_Link
- removed link J3_R_Link
- removed link SL_L_Link
- removed link SL_R_Link
- added link joint1_left_link, mass 0.006; collision mesh filename=package://mygripper_f100_description/meshes/J1_L_Link.STL; visual mesh filename=package://mygripper_f100_description/meshes/J1_L_Link.STL
- added link joint1_right_link, mass 0.006; collision mesh filename=package://mygripper_f100_description/meshes/SL_R_Link.STL; visual mesh filename=package://mygripper_f100_description/meshes/SL_R_Link.STL
- added link joint2_left_link, mass 0.015; collision mesh filename=package://mygripper_f100_description/meshes/J2_L_Link.STL; visual mesh filename=package://mygripper_f100_description/meshes/J2_L_Link.STL
- added link joint2_right_link, mass 0.013; collision mesh filename=package://mygripper_f100_description/meshes/J2_R_Link.STL; visual mesh filename=package://mygripper_f100_description/meshes/J2_R_Link.STL
- added link joint3_left_link, mass 0.017; collision mesh filename=package://mygripper_f100_description/meshes/J3_L_Link.STL; visual mesh filename=package://mygripper_f100_description/meshes/J3_L_Link.STL
- added link joint3_right_link, mass 0.018; collision mesh filename=package://mygripper_f100_description/meshes/J3_R_Link.STL; visual mesh filename=package://mygripper_f100_description/meshes/J3_R_Link.STL
Joints:
- removed joint J2_L_Joint
- removed joint J2_R_joint
- removed joint J3_L_Joint
- removed joint J3_R_joint
- removed joint SL_Joint
- removed joint SL_R_joint
- added joint joint1_left_joint: type revolute, parent f100_base_link, child joint1_left_link, origin xyz=0.033748 0.043203 0 rpy=0 0 0.00036257, axis 0 0 -1, limit lower=-1.012 upper=1.012 effort=0 velocity=0, mimic joint=joint2_left_joint multiplier=1 offset=0
- added joint joint1_right_joint: type revolute, parent f100_base_link, child joint1_right_link, origin xyz=0.033748 -0.045581 0 rpy=0 0 0, axis 0 0 -1, limit lower=-1.012 upper=1.012 effort=0 velocity=0, mimic joint=joint2_left_joint multiplier=-1 offset=0
- added joint joint2_left_joint: type revolute, parent f100_base_link, child joint2_left_link, origin xyz=0.056064 0.017111 0 rpy=0 0 0.00036257, axis 0 0 -1, limit lower=-1.012 upper=0 effort=0 velocity=0
- added joint joint2_right_joint: type revolute, parent f100_base_link, child joint2_right_link, origin xyz=0.056064 -0.019509 0 rpy=0 0 0, axis 0 0 -1, limit lower=-1.012 upper=1.012 effort=0 velocity=0, mimic joint=joint2_left_joint multiplier=-1 offset=0
- added joint joint3_left_joint: type revolute, parent joint2_left_link, child joint3_left_link, origin xyz=0.059996 -0.0097778 -0.0005 rpy=0 0 0, axis 0 0 -1, limit lower=-1.012 upper=1.012 effort=0 velocity=0, mimic joint=joint2_left_joint multiplier=-1 offset=0
- added joint joint3_right_joint: type revolute, parent joint2_right_link, child joint3_right_link, origin xyz=0.06 0.009756 0 rpy=0 0 0, axis 0 0 -1, limit lower=-1.012 upper=1.012 effort=0 velocity=0, mimic joint=joint2_left_joint multiplier=1 offset=0

Commit message: fix(mygripper_f100_description): fix the incorrect link

File: robots_description/mygripper_f100_description/urdf/mygripper_f100.urdf (robot description, URDF)
Before this commit: robot mygripper_f100, 7 links, 6 joints
Links:
- link joint1_right_link: geometry collision mesh filename=package://mygripper_f100_description/meshes/J1_R_Link.STL; visual mesh filename=package://mygripper_f100_description/meshes/J1_R_Link.STL
