Commit message: feat(tutorials): add Pro 450 Tutorial 9 pick-place examples

File: USD/sim_450_f100/config/450_f100.urdf (robot description, URDF)
Before this commit: robot mycobot_pro450, 14 links, 13 joints
Links:
- added link tcp, mass 0.001
Joints:
- added joint tcp_joint: type fixed, parent f100_base_link, child tcp, origin xyz=0 0 0 rpy=0 1.57079632679 0
- joint joint1_left_joint: limit lower=-1.01229097 upper=1.01229097 effort=0 velocity=0 -> lower=-1.01229097 upper=1.01229097 effort=0 velocity=1.0
- joint joint1_right_joint: limit lower=-1.01229097 upper=1.01229097 effort=0 velocity=0 -> lower=-1.01229097 upper=1.01229097 effort=0 velocity=1.0
- joint joint2_left_joint: limit lower=-1.01229097 upper=0 effort=0 velocity=0 -> lower=-1.01229097 upper=0 effort=0 velocity=1.0
- joint joint2_right_joint: limit lower=-1.01229097 upper=1.01229097 effort=0 velocity=0 -> lower=-1.01229097 upper=1.01229097 effort=0 velocity=1.0
- joint joint3_left_joint: limit lower=-1.01229097 upper=1.01229097 effort=0 velocity=0 -> lower=-1.01229097 upper=1.01229097 effort=0 velocity=1.0
- joint joint3_right_joint: limit lower=-1.01229097 upper=1.01229097 effort=0 velocity=0 -> lower=-1.01229097 upper=1.01229097 effort=0 velocity=1.0
